File: MultiVIb_Mareks/M_Krisjanis_MultiVibe/N_Krisjanis_MultiVibe.sch (KiCad schematic (older format))
At the start: 10 parts, among them U1 SSM2210

Commit message: 2_md_Power_supply
Parts:
- U1: symbol apzimejums0:SSM2210 -> N_Krisjanis_MultiVibe-rescue:SSM2210-apzimejums0
Changed lines of the file:
@@
 Connection ~ 3800 1550
 $Comp
-L apzimejums0:SSM2210 U1
+L N_Krisjanis_MultiVibe-rescue:SSM2210-apzimejums0 U1
 U 1 1 5F7E0DC8
 P 4300 3775
