File: Battery_Mareks/Battery_Mareks.sch (KiCad schematic (older format))
At the start: 1 part

Commit message: 4 md par baterijām un to lodlaukumiem
Parts:
- BT1: footprint Battery_Holder_:SMTU2032 -> Battery_Holder_:BC-2001
Changed lines of the file:
@@
 F 0 "BT1" H 4793 3796 50  0000 L CNN
 F 1 "Battery_Cell" H 4793 3705 50  0000 L CNN
-F 2 "Battery_Holder_:SMTU2032" V 4675 3760 50  0001 C CNN
+F 2 "Battery_Holder_:BC-2001" V 4675 3760 50  0001 C CNN
 F 3 "~" V 4675 3760 50  0001 C CNN
 	1    4675 3700
