File: Single_Tranzistor_AMP/Single_Tranzistor_AMP.sch (KiCad schematic (older format))
At the start: 12 parts, among them J1 Screw_Terminal_01x03, Q1 BC547, Q2 BC557

Commit message: majasdarbs par celinu trasesanu
Connections:
- net GNDREF: now reaches BZ1.2 (+), C2.2, J1.1 (Pin_1), R2.2, R4.2
Changed lines of the file:
@@
 	6600 3550 5975 3550
 Connection ~ 5975 3550
+$Comp
+L power:GNDREF #PWR01
+U 1 1 5FC95636
+P 4450 5600
+F 0 "#PWR01" H 4450 5350 50  0001 C CNN
+F 1 "GNDREF" H 4455 5427 50  0000 C CNN
+F 2 "" H 4450 5600 50  0001 C CNN
+F 3 "" H 4450 5600 50  0001 C CNN
+	1    4450 5600
+	1    0    0    -1
+$EndComp
+Connection ~ 4450 5600
 $EndSCHEMATC
